Commit message: Fix xml formatting

File: kortex_description/robots/kortex_robot.xacro (robot description, xacro)
@@ -65,23 +65,23 @@
     <!-- Include and load the gripper if defined -->
     <xacro:unless value="${not gripper}">
-    <!-- Define an updated "last_arm_link" to correctly offset the F/T-->
-    <xacro:property name="sensor_height_offset" value="0.06"/>
-      <link name="${prefix}tool_frame"/>
-      <joint name="${prefix}tool_frame_joint" type="fixed">
-        <origin xyz="0 0 ${sensor_height_offset}" rpy="0 0 0" />
-        <parent link="${prefix}${last_arm_link}" />
-        <child link="${prefix}tool_frame" />
-        <axis xyz="0 0 0" />
-      </joint>
+      <!-- Define an updated "last_arm_link" to correctly offset the F/T-->
+      <xacro:property name="sensor_height_offset" value="0.06"/>
+        <link name="${prefix}tool_frame"/>
+        <joint name="${prefix}tool_frame_joint" type="fixed">
+          <origin xyz="0 0 ${sensor_height_offset}" rpy="0 0 0" />
+          <parent link="${prefix}${last_arm_link}" />
+          <child link="${prefix}tool_frame" />
+          <axis xyz="0 0 0" />
+        </joint>
       <xacro:include filename="$(find kortex_description)/grippers/${gripper}/urdf/${gripper}_macro.xacro" />
-      <!-- last_arm_link is defined in "$(find kortex_description)/arms/${arm}/urdf/${arm}_macro.xacro" -->
-     <xacro:if value="${fake_sensor_commands}">
-        <xacro:load_gripper
-          parent="${prefix}${last_arm_link}"
-          prefix="${prefix}"
-          use_fake_hardware="${use_fake_hardware}"
-          fake_sensor_commands="${fake_sensor_commands}"
-          sim_ignition="${sim_ignition}"
-          sim_isaac="${sim_isaac}"/>
+        <!-- last_arm_link is defined in "$(find kortex_description)/arms/${arm}/urdf/${arm}_macro.xacro" -->
+      <xacro:if value="${fake_sensor_commands}">
+          <xacro:load_gripper
+            parent="${prefix}${last_arm_link}"
+            prefix="${prefix}"
+            use_fake_hardware="${use_fake_hardware}"
+            fake_sensor_commands="${fake_sensor_commands}"
+            sim_ignition="${sim_ignition}"
+            sim_isaac="${sim_isaac}"/>
       </xacro:if>
       <xacro:unless value="${fake_sensor_commands}">
