Commit message: Update xacro & configs for admittance controller

File: kortex_description/arms/gen3/7dof/urdf/kortex.ros2_control.xacro (robot description, xacro)
@@ -161,4 +161,28 @@
         <state_interface name="effort"/>
       </joint>
+      <!-- Correctly load the admittance controller -->
+      <sensor name="${tf_prefix}ati_ft_sensor">
+        <state_interface name="force.x"/>
+        <state_interface name="force.y"/>
+        <state_interface name="force.z"/>
+        <state_interface name="torque.x"/>
+        <state_interface name="torque.y"/>
+        <state_interface name="torque.z"/>
+      </sensor>
+        <!-- Correctly use F/T wrench with the fake controller  -->
+      <joint name="ati_ft_sensor">
+        <command_interface name="force.x"/>
+        <command_interface name="force.y"/>
+        <command_interface name="force.z"/>
+        <command_interface name="torque.x"/>
+        <command_interface name="torque.y"/>
+        <command_interface name="torque.z"/>
+        <state_interface name="force.x"/>
+        <state_interface name="force.y"/>
+        <state_interface name="force.z"/>
+        <state_interface name="torque.x"/>
+        <state_interface name="torque.y"/>
+        <state_interface name="torque.z"/>
+      </joint>
       <xacro:if value="${use_internal_bus_gripper_comm}">
         <joint name="${prefix}${gripper_joint_name}">

Commit message: Dynamically load the ati hardware interface for admittance control

File: kortex_description/arms/gen3/7dof/urdf/kortex.ros2_control.xacro (robot description, xacro)
@@ -161,6 +161,6 @@
         <state_interface name="effort"/>
       </joint>
-      <!-- Correctly load the admittance controller -->
-      <sensor name="${tf_prefix}ati_ft_sensor">
+      <!-- Load the admittance controller -->
+      <sensor name="${prefix}tcp_fts_sensor">
         <state_interface name="force.x"/>
         <state_interface name="force.y"/>
@@ -170,19 +170,21 @@
         <state_interface name="torque.z"/>
       </sensor>
-        <!-- Correctly use F/T wrench with the fake controller  -->
-      <joint name="ati_ft_sensor">
-        <command_interface name="force.x"/>
-        <command_interface name="force.y"/>
-        <command_interface name="force.z"/>
-        <command_interface name="torque.x"/>
-        <command_interface name="torque.y"/>
-        <command_interface name="torque.z"/>
-        <state_interface name="force.x"/>
-        <state_interface name="force.y"/>
-        <state_interface name="force.z"/>
-        <state_interface name="torque.x"/>
-        <state_interface name="torque.y"/>
-        <state_interface name="torque.z"/>
-      </joint>
+        <!-- Correctly use the F/T wrench with the fake controller  -->
+      <xacro:if value="${use_fake_hardware}">
+        <joint name="${prefix}tcp_fts_sensor">
+          <command_interface name="force.x"/>
+          <command_interface name="force.y"/>
+          <command_interface name="force.z"/>
+          <command_interface name="torque.x"/>
+          <command_interface name="torque.y"/>
+          <command_interface name="torque.z"/>
+          <state_interface name="force.x"/>
+          <state_interface name="force.y"/>
+          <state_interface name="force.z"/>
+          <state_interface name="torque.x"/>
+          <state_interface name="torque.y"/>
+          <state_interface name="torque.z"/>
+        </joint>
+      </xacro:if>
       <xacro:if value="${use_internal_bus_gripper_comm}">
         <joint name="${prefix}${gripper_joint_name}">
@@ -194,3 +196,23 @@
     </ros2_control>
   </xacro:macro>
+  <!-- Net FT args -->
+  <xacro:arg name="sensor_type" default="ati"/>
+  <xacro:arg name="ip_address" default="192.168.1.84"/>
+  <xacro:arg name="rdt_sampling_rate" default="500"/>
+  <xacro:arg name="internal_filter_rate" default="false"/>
+  <xacro:arg name="use_hardware_biasing" default="false"/>
+  <xacro:arg name="prefix" default=""/>
+  <!-- Import netft macros -->
+    <xacro:include filename="$(find net_ft_description)/urdf/net_ft_sensor_macro.urdf.xacro" />
+  <!-- Force Sensor -->
+  <xacro:net_ft_sensor parent="end_effector_link"
+  prefix="$(arg prefix)"
+  ip_address="$(arg ip_address)"
+  rdt_sampling_rate="$(arg rdt_sampling_rate)"
+  sensor_type="$(arg sensor_type)"
+  internal_filter_rate="$(arg internal_filter_rate)"
+  use_hardware_biasing="$(arg use_hardware_biasing)">
+  <!-- Create link fixed to the "world" -->
+  <link name="world" />
+  </xacro:net_ft_sensor>
 </robot>

Commit message: Load F/T based on fake_sensor_commands arg

File: kortex_description/arms/gen3/7dof/urdf/kortex.ros2_control.xacro (robot description, xacro)
@@ -200,19 +200,21 @@
   <xacro:arg name="ip_address" default="192.168.1.84"/>
   <xacro:arg name="rdt_sampling_rate" default="500"/>
-  <xacro:arg name="internal_filter_rate" default="false"/>
+  <xacro:arg name="internal_filter_rate" default="0"/>
   <xacro:arg name="use_hardware_biasing" default="false"/>
   <xacro:arg name="prefix" default=""/>
-  <!-- Import netft macros -->
-    <xacro:include filename="$(find net_ft_description)/urdf/net_ft_sensor_macro.urdf.xacro" />
-  <!-- Force Sensor -->
-  <xacro:net_ft_sensor parent="end_effector_link"
-  prefix="$(arg prefix)"
-  ip_address="$(arg ip_address)"
-  rdt_sampling_rate="$(arg rdt_sampling_rate)"
-  sensor_type="$(arg sensor_type)"
-  internal_filter_rate="$(arg internal_filter_rate)"
-  use_hardware_biasing="$(arg use_hardware_biasing)">
-  <!-- Create link fixed to the "world" -->
-  <link name="world" />
-  </xacro:net_ft_sensor>
+  <!-- Import Net FT  macros -->
+  <xacro:include filename="$(find net_ft_description)/urdf/net_ft_sensor_macro.urdf.xacro" />
+  <!-- Force Sensor: Allow the F/T sensor data to be available to both the sim and real hardware -->
+  <xacro:unless value="${fake_sensor_commands}">
+    <xacro:net_ft_sensor parent="end_effector_link"
+      prefix="$(arg prefix)"
+      ip_address="$(arg ip_address)"
+      rdt_sampling_rate="$(arg rdt_sampling_rate)"
+      sensor_type="$(arg sensor_type)"
+      internal_filter_rate="$(arg internal_filter_rate)"
+      use_hardware_biasing="$(arg use_hardware_biasing)">
+      <!-- Create link fixed to the "world" -->
+      <link name="world" />
+    </xacro:net_ft_sensor>
+  </xacro:unless>
 </robot>

Commit message: Temp NetFT fix

File: kortex_description/arms/gen3/7dof/urdf/kortex.ros2_control.xacro (robot description, xacro)
@@ -196,4 +196,13 @@
     </ros2_control>
   </xacro:macro>
+<!-- Define an updated "tool_frame1" relative to the "tool_frame" to correctly offset the F/T-->
+    <xacro:property name="frame_offset" value="-0.004"/>
+      <link name="${prefix}tool_frame1"/>
+      <joint name="${prefix}tool_frame_joint1" type="fixed">
+        <origin xyz="0 0 ${frame_offset}" rpy="0 0 0" />
+        <parent link="tool_frame" />
+        <child link="tool_frame1" />
+        <axis xyz="0 0 0" />
+      </joint>
   <!-- Net FT args -->
   <xacro:arg name="sensor_type" default="ati"/>
@@ -207,5 +216,6 @@
   <!-- Force Sensor: Allow the F/T sensor data to be available to both the sim and real hardware -->
   <xacro:unless value="${fake_sensor_commands}">
-    <xacro:net_ft_sensor parent="end_effector_link"
+    <xacro:net_ft_sensor
+      parent="tool_frame1"
       prefix="$(arg prefix)"
       ip_address="$(arg ip_address)"

File: kortex_description/robots/kortex_robot.xacro (robot description, xacro)
@@ -65,13 +65,33 @@
     <!-- Include and load the gripper if defined -->
     <xacro:unless value="${not gripper}">
+    <!-- Define an updated "last_arm_link" to correctly offset the F/T-->
+    <xacro:property name="sensor_height_offset" value="0.06"/>
+      <link name="${prefix}tool_frame"/>
+      <joint name="${prefix}tool_frame_joint" type="fixed">
+        <origin xyz="0 0 ${sensor_height_offset}" rpy="0 0 0" />
+        <parent link="${prefix}${last_arm_link}" />
+        <child link="${prefix}tool_frame" />
+        <axis xyz="0 0 0" />
+      </joint>
       <xacro:include filename="$(find kortex_description)/grippers/${gripper}/urdf/${gripper}_macro.xacro" />
       <!-- last_arm_link is defined in "$(find kortex_description)/arms/${arm}/urdf/${arm}_macro.xacro" -->
-      <xacro:load_gripper
-        parent="${prefix}${last_arm_link}"
-        prefix="${prefix}"
-        use_fake_hardware="${use_fake_hardware}"
-        fake_sensor_commands="${fake_sensor_commands}"
-        sim_ignition="${sim_ignition}"
-        sim_isaac="${sim_isaac}"/>
+     <xacro:if value="${fake_sensor_commands}">
+        <xacro:load_gripper
+          parent="${prefix}${last_arm_link}"
+          prefix="${prefix}"
+          use_fake_hardware="${use_fake_hardware}"
+          fake_sensor_commands="${fake_sensor_commands}"
+          sim_ignition="${sim_ignition}"
+          sim_isaac="${sim_isaac}"/>
+      </xacro:if>
+      <xacro:unless value="${fake_sensor_commands}">
+        <xacro:load_gripper
+          parent="${prefix}tool_frame"
+          prefix="${prefix}"
+          use_fake_hardware="${use_fake_hardware}"
+          fake_sensor_commands="${fake_sensor_commands}"
+          sim_ignition="${sim_ignition}"
+          sim_isaac="${sim_isaac}"/>
+      </xacro:unless>
     </xacro:unless>
   </xacro:macro>

Commit message: Add controllers (#1)
* Update README for humble

* Add admittance controller

* Update xacro & configs for admittance controller

* Dynamically load the ati hardware interface for admittance control

* Load F/T based on fake_sensor_commands arg

* Update README to reflect F/T launch methods

File: kortex_description/arms/gen3/7dof/urdf/kortex.ros2_control.xacro (robot description, xacro)
@@ -161,4 +161,30 @@
         <state_interface name="effort"/>
       </joint>
+      <!-- Load the admittance controller -->
+      <sensor name="${prefix}tcp_fts_sensor">
+        <state_interface name="force.x"/>
+        <state_interface name="force.y"/>
+        <state_interface name="force.z"/>
+        <state_interface name="torque.x"/>
+        <state_interface name="torque.y"/>
+        <state_interface name="torque.z"/>
+      </sensor>
+        <!-- Correctly use the F/T wrench with the fake controller  -->
+      <xacro:if value="${use_fake_hardware}">
+        <joint name="${prefix}tcp_fts_sensor">
+          <command_interface name="force.x"/>
+          <command_interface name="force.y"/>
+          <command_interface name="force.z"/>
+          <command_interface name="torque.x"/>
+          <command_interface name="torque.y"/>
+          <command_interface name="torque.z"/>
+          <state_interface name="force.x"/>
+          <state_interface name="force.y"/>
+          <state_interface name="force.z"/>
+          <state_interface name="torque.x"/>
+          <state_interface name="torque.y"/>
+          <state_interface name="torque.z"/>
+        </joint>
+      </xacro:if>
       <xacro:if value="${use_internal_bus_gripper_comm}">
         <joint name="${prefix}${gripper_joint_name}">
@@ -170,3 +196,25 @@
     </ros2_control>
   </xacro:macro>
+  <!-- Net FT args -->
+  <xacro:arg name="sensor_type" default="ati"/>
+  <xacro:arg name="ip_address" default="192.168.1.84"/>
+  <xacro:arg name="rdt_sampling_rate" default="500"/>
+  <xacro:arg name="internal_filter_rate" default="0"/>
+  <xacro:arg name="use_hardware_biasing" default="false"/>
+  <xacro:arg name="prefix" default=""/>
+  <!-- Import Net FT  macros -->
+  <xacro:include filename="$(find net_ft_description)/urdf/net_ft_sensor_macro.urdf.xacro" />
+  <!-- Force Sensor: Allow the F/T sensor data to be available to both the sim and real hardware -->
+  <xacro:unless value="${fake_sensor_commands}">
+    <xacro:net_ft_sensor parent="end_effector_link"
+      prefix="$(arg prefix)"
+      ip_address="$(arg ip_address)"
+      rdt_sampling_rate="$(arg rdt_sampling_rate)"
+      sensor_type="$(arg sensor_type)"
+      internal_filter_rate="$(arg internal_filter_rate)"
+      use_hardware_biasing="$(arg use_hardware_biasing)">
+      <!-- Create link fixed to the "world" -->
+      <link name="world" />
+    </xacro:net_ft_sensor>
+  </xacro:unless>
 </robot>
