Commit message: bringing back the gripper

File: kortex_description/arms/gen3/7dof/urdf/gen3_macro.xacro (robot description, xacro)
@@ -2,5 +2,6 @@
 <robot name="gen3_arm" xmlns:xacro="http://ros.org/wiki/xacro">
   <!-- Propagate last link name information because it is the gripper's parent link -->
-  <xacro:property name="last_arm_link" value="end_effector_link"/>
+  <!-- Commenting out the line below to prevent an override -->
+  <!-- <xacro:property name="last_arm_link" value="end_effector_link"/> -->
   <xacro:property name="PI" value="3.1415926535897931"/>
   <xacro:macro name="load_arm" params="

File: kortex_description/robots/kortex_robot.xacro (robot description, xacro)
@@ -26,4 +26,5 @@
     isaac_joint_states:=/isaac_joint_states
     use_external_cable:=false
+    last_arm_link:=end_effector_link
     initial_positions:=${dict(joint_1=0.0,joint_2=0.0,joint_3=0.0,joint_4=0.0,joint_5=0.0,joint_6=0.0,joint_7=0.0)}
     gripper_max_velocity:=100.0

Commit message: Adding a collision box to the camera for safety

File: kortex_description/arms/gen3/7dof/urdf/gen3_macro.xacro (robot description, xacro)
@@ -375,4 +375,10 @@
         </geometry>
       </collision>
+      <collision>
+        <origin xyz="0.0 -0.03 -0.065" rpy="0 0 0"/>
+        <geometry>
+          <box size="0.12 0.12 0.05"/>
+        </geometry>
+      </collision>
     </link>
     </xacro:if>
@@ -397,4 +403,10 @@
         <geometry>
           <mesh filename="file://$(find kortex_description)/arms/gen3/${dof}dof/meshes/bracelet_no_vision_link.dae" />
+        </geometry>
+      </collision>
+       <collision>
+        <origin xyz="0.03 0.00 0.01" rpy="0 0 0"/>
+        <geometry>
+          <box size="0.4 0.4 0.4"/>
         </geometry>
       </collision>

Commit message: Adding a collision box to make hardware usage safer for the camera

File: kortex_description/arms/gen3/7dof/urdf/gen3_macro.xacro (robot description, xacro)
@@ -1,3 +1,4 @@
 <?xml version="1.0"?>
+#gen3_macro.xacro
 <robot name="gen3_arm" xmlns:xacro="http://ros.org/wiki/xacro">
   <!-- Propagate last link name information because it is the gripper's parent link -->
